Commit message: Fixes

File: pegasus_base/urdf/pegasus_mini.urdf (robot description, URDF)
Before this commit: robot pegasus_mini, 6 links, 5 joints
Links:
- removed link backcastor
Joints:
- removed joint backcastor_joint
- joint frontcastor_joint: origin xyz=0 0 0 rpy=0 0 0 -> xyz=0.194 0 -0.025 rpy=0 0 0
- joint laser_joint: origin xyz=0.16688 -0.001 0.1019 rpy=0 0 3.1415 -> xyz=0.24679 0 0.09 rpy=0 0 3.1415
- joint leftwheel_joint: origin xyz=0 0.124 0 rpy=0 0 0 -> xyz=0 0.1279 0 rpy=0 0 0
- joint rightwheel_joint: origin xyz=0 -0.123 0 rpy=0 0 0 -> xyz=0 -0.1279 0 rpy=0 0 0

Commit message: Apriltags Additions

File: pegasus_base/urdf/pegasus_mini.urdf (robot description, URDF)
Before this commit: robot pegasus_mini, 5 links, 4 joints
Links:
- added link camera, mass 0.232013920708616; collision cylinder length=0.02 radius=0.0375; visual box size=0.001 0.001 0.001
Joints:
- added joint camera_joint: type fixed, parent base_link, child camera, origin xyz=0.3 0 0.098 rpy=0 0 0, axis 0 1 0

Commit message: Changes

File: pegasus_base/urdf/pegasus_mini.urdf (robot description, URDF)
Before this commit: robot pegasus_mini, 6 links, 5 joints
Joints:
- joint camera_joint: origin xyz=0.3 0 0.098 rpy=0 0 0 -> xyz=0.3 0 0.098 rpy=-1.5707 0 -1.5707

Commit message: Changes

File: pegasus_base/urdf/pegasus_mini.urdf (robot description, URDF)
Before this commit: robot pegasus_mini, 6 links, 5 joints
Joints:
- joint laser_joint: origin xyz=0.24679 0 0.098 rpy=0 0 3.1415 -> xyz=0.24679 0 0.098 rpy=0 0 3.14159

Commit message: Updates

File: pegasus_base/urdf/pegasus_mini.urdf (robot description, URDF)
Before this commit: robot pegasus_mini, 6 links, 5 joints
Joints:
- joint camera_joint: origin xyz=0.3 0 0.098 rpy=-1.5707 0 -1.5707 -> xyz=0.34 0 0.098 rpy=-1.5707 0 -1.5707

Commit message: Updates

File: pegasus_base/urdf/pegasus_mini.urdf (robot description, URDF)
Before this commit: robot pegasus_mini, 6 links, 5 joints
Links:
- added link imu_link, mass 0.0; collision box size=0.001 0.001 0.001; visual box size=0.001 0.001 0.001
Joints:
- added joint imu_joint: type fixed, parent base_link, child imu_link, origin xyz=0 0 00 rpy=0 0 0, axis 0 1 0

Commit message: Final Changes

File: pegasus_base/urdf/pegasus_mini.urdf (robot description, URDF)
Before this commit: robot pegasus_mini, 7 links, 6 joints
Joints:
- joint camera_joint: origin xyz=0.34 0 0.098 rpy=-1.5707 0 -1.5707 -> xyz=0.33 0 0.098 rpy=-1.57079 0 -1.57079
